File: project_files/encoder_buttons.kicad_pcb (KiCad board)
At the start: 2 copper layers, 63.5 x 25.4 mm, 39 parts, among them J1 UPPER, SW1 A, SW3 B, SW4 A, SW5 C, SW6 B, SW7 C, SW8 EC11, U1 74HC14, U2 74HC14

Commit message: Finalized and rendered
Parts:
- added REF**: OSHW-Logo2_9.8x8mm_SilkScreen, Symbol:OSHW-Logo2_9.8x8mm_SilkScreen, B.Cu at (118.7, 85.7)
- moved D6 0.85 mm to (121.4, 77.7)
- moved D2 0.83 mm to (121.4, 93.7)
- moved D4 0.80 mm to (121.4, 86.1)
- moved C5 0.64 mm to (101.6, 92.1)
- moved R11 0.64 mm to (97.8, 92.1)
- moved R5 0.64 mm to (97.8, 81.9)
- moved R6 0.64 mm to (122.6, 81.9)
- moved R9 0.64 mm to (97.8, 90.2)
- moved C3 0.63 mm to (101.6, 83.8)
- moved R10 0.63 mm to (122.6, 73.7)
- moved R7 0.63 mm to (97.8, 83.8)
- moved D1 0.47 mm to (98.8, 77.7)
- moved D3 0.38 mm to (98.8, 86.0)
- moved D5 0.38 mm to (98.8, 94.2)
- turned C6 to 180 degrees
Routing:
- net VCC: track 2.98 -> 99.4 mm, vias 3 -> 6
- net Net-(D2-A): track 0.00 -> 24.3 mm
- net Net-(D3-A): track 0.00 -> 15.8 mm
- net Net-(D1-A): track 0.00 -> 15.0 mm
- net Net-(D5-A): track 0.00 -> 15.0 mm
- net /ENC_A: track 3.79 -> 18.3 mm
- net /BUT_C: track 5.66 -> 19.1 mm
- net /BUT_B: track 5.66 -> 18.8 mm
- net /ENC_C: track 3.78 -> 16.6 mm
- net /BUT_A: track 6.72 -> 18.8 mm
- net /ENC_B: track 2.47 -> 14.1 mm
- net Net-(D6-A): track 0.00 -> 9.80 mm
- net Net-(D4-A): track 0.00 -> 8.12 mm
- net GND: track 0.00 -> 1.40 mm, vias 0 -> 37
Other:
- board text added: "A"
- board text added: "A_{B}"
- board text added: "A_{EN}"
- board text added: "B"
- board text added: "BUT-A"
- board text added: "BUT-B"
- board text added: "BUT-C"
- board text added: "B_{B}"
- board text added: "B_{EN}"
- board text added: "Buttons and Encoder module with hardware debouncing"
- board text added: "C"
- board text added: "C_{B}"
- board text added: "C_{EN}"
- board text added: "ENC-A"
- board text added: "ENC-B"
- board text added: "ENC-C"
- board text added: "Gnd"
- board text added: "Vcc"
- board text removed: "BUT_A"
- board text removed: "BUT_B"
- board text removed: "BUT_C"
- board text removed: "ENC_A"
- board text removed: "ENC_B"
- board text removed: "ENC_C"
